File: fx-mg100dfx.kicad_pcb (KiCad board)
At the start: 4 copper layers, 56.2 x 66 mm, 71 parts, among them J1 DAUGHTERBOARD IN, J2 DAUGHERBOARD OUT, J3 PPCB STANDARD, J4 9V IN, J5 GND IN, J6 GND IN, J7 GND IN, Q1 BC547C, SW1 OD1/OD2, U1 JRC4558, U2 JRC4558

Commit message: Checkpoint PCB (description diffs)
Parts:
- SW1: value OD1/OD2 -> ON-ON
Changed lines of the file:
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@@
 			)
 		)
-		(property "Description" "Unpolarized capacitor, small symbol - X7R MLCC"
+		(property "Description" "Electrolytic Bulk Capacitor"
 			(at 0 0 90)
 			(layer "F.Fab")
@@
 			)
 		)
+		(property "Notes" "25V min, 35V better"
+			(at -83.794888 177.5 0)
+			(layer "F.SilkS")
+			(hide yes)
+			(effects
+				(font
+					(size 1.27 1.27)
+				)
+			)
+		)
 		(property ki_fp_filters "C_*")
 		(sheetname "/")
 		(sheetfile "fx-mg100dfx.kicad_sch")
-		(units
-			(unit
-				(name "A")
-				(pins "1" "2")
-			)
-		)
 		(attr through_hole)
 		(duplicate_pad_numbers_are_jumpers no)
@@
 			)
 		)
-		(property "Description" "Polarized capacitor, small US symbol"
+		(property "Description" "Electrolytic Bulk Capacitor"
 			(at 0 0 90)
 			(layer "F.Fab")
@@
 			)
 		)
+		(property "Notes" "25V min, 35V better"
+			(at -109.918071 171.58906 0)
+			(layer "F.SilkS")
+			(hide yes)
+			(effects
+				(font
+					(size 1.27 1.27)
+				)
+			)
+		)
 		(property ki_fp_filters "CP_*")
 		(sheetname "/")
 		(sheetfile "fx-mg100dfx.kicad_sch")
-		(units
-			(unit
-				(name "A")
-				(pins "1" "2")
-			)
-		)
 		(attr through_hole)
 		(duplicate_pad_numbers_are_jumpers no)
@@
 			)
 		)
-		(property "Description" "Polarized capacitor, small US symbol"
+		(property "Description" "Electrolytic Bulk Capacitor"
 			(at 0 0 90)
 			(layer "F.Fab")
@@
 			)
 		)
+		(property "Notes" "25V min, 35V better - Base cap for multiplier"
+			(at -109.918071 164.78897 0)
+			(layer "F.SilkS")
+			(hide yes)
+			(effects
+				(font
+					(size 1.27 1.27)
+				)
+			)
+		)
 		(property ki_fp_filters "CP_*")
 		(sheetname "/")
 		(sheetfile "fx-mg100dfx.kicad_sch")
-		(units
-			(unit
-				(name "A")
-				(pins "1" "2")
-			)
-		)
 		(attr through_hole)
 		(duplicate_pad_numbers_are_jumpers no)
@@
 			)
 		)
+		(property "Notes" "Cap Multiplier Base (See Note)"
+			(at 156.913912 109.467584 0)
+			(layer "F.SilkS")
+			(hide yes)
+			(effects
+				(font
+					(size 1.27 1.27)
+				)
+			)
+		)
 		(property ki_fp_filters "R_*")
 		(sheetname "/")
 		(sheetfile "fx-mg100dfx.kicad_sch")
-		(units
-			(unit
-				(name "A")
-				(pins "1" "2")
-			)
-		)
 		(attr through_hole)
 		(duplicate_pad_numbers_are_jumpers no)
@@
 			)
 		)
-		(property "Value" "OD1/OD2"
-			(at 2.55 0.03581 90)
+		(property "Value" "ON-ON"
+			(at -4 0.03581 90)
 			(layer "F.SilkS")
 			(effects
@@
 			(at 0 0 0)
 			(unlocked yes)
+			(layer "F.Fab")
+			(hide yes)
+			(effects
+				(font
+					(size 1 1)
+					(thickness 0.15)
+				)
+			)
+		)
+		(property "Control" "OD1/OD2"
+			(at 0 0 0)
+			(unlocked yes)

Commit message: fx-mg100dfx 0.3 fab outputs (g1)
Changed lines of the file:
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@@
 	(paper "A4")
 	(title_block
-		(title "MG100DFX")
-		(rev "0.3TH")
+		(title "MG100DFX-TH")
+		(rev "0.3")
 	)
 	(layers

Commit message: fx-mg100dfx 0.4 fab outputs (g3)
Parts:
- R11: value 1.5k -> 1.5K
- R12, R21: value 4.7k -> 4.7K
- R13: value 3.3k -> 3.3K
- R16: value 33k -> 33K
- R17: value 47k -> 47K
- R20: value 1.8k -> 1.8K
- R4: value 15k -> 4.7K
- R7: value 22k -> 22K
- RV1: value B1M -> A1M
- SW1: value ON-ON -> OD1/OD2
Changed lines of the file:
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@@
 	(title_block
 		(title "MG100DFX-TH")
-		(rev "0.3")
+		(rev "0.4")
 	)
 	(layers
@@
 			)
 		)
-		(property "Value" "1.5k"
+		(property "Value" "1.5K"
 			(at 3.81 0 0)
 			(layer "F.SilkS")
@@
 			)
 		)
-		(property "Description" "Electrolytic Bulk Capacitor"
+		(property "Description" "Unpolarized capacitor, small symbol - X7R MLCC"
 			(at 0 0 90)
 			(layer "F.Fab")
@@
 			)
 		)
-		(property "Notes" "25V min, 35V better"
-			(at -83.794888 177.5 0)
-			(layer "F.SilkS")
-			(hide yes)
-			(effects
-				(font
-					(size 1.27 1.27)
-				)
-			)
-		)
 		(property ki_fp_filters "C_*")
 		(sheetname "/")
 		(sheetfile "fx-mg100dfx.kicad_sch")
+		(units
+			(unit
+				(name "A")
+				(pins "1" "2")
+			)
+		)
 		(attr through_hole)
 		(duplicate_pad_numbers_are_jumpers no)
@@
 			)
 		)
-		(property "Description" "Electrolytic Bulk Capacitor"
+		(property "Description" "Polarized capacitor, small US symbol"
 			(at 0 0 90)
 			(layer "F.Fab")
@@
 			)
 		)
-		(property "Notes" "25V min, 35V better"
-			(at -109.918071 171.58906 0)
-			(layer "F.SilkS")
-			(hide yes)
-			(effects
-				(font
-					(size 1.27 1.27)
-				)
-			)
-		)
 		(property ki_fp_filters "CP_*")
 		(sheetname "/")
 		(sheetfile "fx-mg100dfx.kicad_sch")
+		(units
+			(unit
+				(name "A")
+				(pins "1" "2")
+			)
+		)
 		(attr through_hole)
 		(duplicate_pad_numbers_are_jumpers no)
@@
 			)
 		)
-		(property "Description" "Electrolytic Bulk Capacitor"
+		(property "Description" "Polarized capacitor, small US symbol"
 			(at 0 0 90)
 			(layer "F.Fab")
@@
 			)
 		)
-		(property "Notes" "25V min, 35V better - Base cap for multiplier"
-			(at -109.918071 164.78897 0)
-			(layer "F.SilkS")
-			(hide yes)
-			(effects
-				(font
-					(size 1.27 1.27)
-				)
-			)
-		)
 		(property ki_fp_filters "CP_*")
 		(sheetname "/")
 		(sheetfile "fx-mg100dfx.kicad_sch")
+		(units
+			(unit
+				(name "A")
+				(pins "1" "2")
+			)
+		)
 		(attr through_hole)
 		(duplicate_pad_numbers_are_jumpers no)
@@
 			)
 		)
-		(property "Value" "47k"
+		(property "Value" "47K"
 			(at 3.81 0 0)
 			(layer "F.SilkS")
@@
 			)
 		)
-		(property "Value" "33k"
+		(property "Value" "33K"
 			(at 3.81 0 0)
 			(layer "F.SilkS")
@@
 			)
 		)
-		(property "Notes" "Cap Multiplier Base (See Note)"
-			(at 156.913912 109.467584 0)
-			(layer "F.SilkS")
-			(hide yes)
-			(effects
-				(font
-					(size 1.27 1.27)
-				)
-			)
-		)
 		(property ki_fp_filters "R_*")
 		(sheetname "/")
 		(sheetfile "fx-mg100dfx.kicad_sch")
+		(units
+			(unit
+				(name "A")
+				(pins "1" "2")
+			)
+		)
 		(attr through_hole)
 		(duplicate_pad_numbers_are_jumpers no)
@@
 			)
 		)
-		(property "Value" "4.7k"
+		(property "Value" "4.7K"
 			(at 3.81 0 0)
 			(layer "F.SilkS")
@@
 			)
 		)
-		(property "Value" "4.7k"
+		(property "Value" "4.7K"
 			(at 3.81 0 0)
 			(layer "F.SilkS")
@@
 			)
 		)
-		(property "Value" "22k"
+		(property "Value" "22K"
 			(at 3.81 0 0)
 			(layer "F.SilkS")
@@
 			)
 		)
-		(property "Value" "1.8k"
+		(property "Value" "1.8K"
 			(at 3.81 0 0)
 			(layer "F.SilkS")
@@
 			)
 		)
-		(property "Value" "15k"
+		(property "Value" "4.7K"
 			(at 3.81 0 0)
 			(layer "F.SilkS")
@@
 			)
 		)
-		(property "Value" "B1M"
+		(property "Value" "A1M"
 			(at -6.604 -2.286 0)
 			(layer "F.SilkS")
@@
 			)
 		)
-		(property "Value" "3.3k"
+		(property "Value" "3.3K"
 			(at 3.81 0 0)
 			(layer "F.SilkS")
@@
 			)
 		)
-		(property "Value" "ON-ON"
+		(property "Value" "OD1/OD2"
 			(at -4 0.03581 90)
 			(layer "F.SilkS")
@@
 			(at 0 0 0)
 			(unlocked yes)
-			(layer "F.Fab")
-			(hide yes)
-			(effects
-				(font
-					(size 1 1)
-					(thickness 0.15)
-				)
-			)
-		)
-		(property "Control" "OD1/OD2"
-			(at 0 0 0)
-			(unlocked yes)
