File: fx-mg100dfx.kicad_sch (KiCad schematic)
At the start: 71 parts, among them J1 DAUGHTERBOARD IN, J2 DAUGHERBOARD OUT, J3 PPCB STANDARD, J4 9V IN, J5 GND IN, J6 GND IN, J7 GND IN, Q1 BC547C, SW1 OD1/OD2, U1 JRC4558, U2 JRC4558

Commit message: fx-mg100dfx 0.3 fab outputs (g1)
Other:
- moved on the sheet: D1

Commit message: fx-mg100dfx 0.4 fab outputs (g3)
Parts:
- R11: value 1.5k -> 1.5K
- R12, R21: value 4.7k -> 4.7K
- R13: value 3.3k -> 3.3K
- R16: value 33k -> 33K
- R17: value 47k -> 47K
- R20: value 1.8k -> 1.8K
- R4: value 15k -> 4.7K
- R7: value 22k -> 22K
- RV1: value B1M -> A1M
Changed lines of the file:
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@@
 			)
 		)
-		(property "Value" "3.3k"
+		(property "Value" "3.3K"
 			(at 163.83 78.994 90)
 			(show_name no)
@@
 			)
 		)
-		(property "Value" "B1M"
+		(property "Value" "A1M"
 			(at 135.382 102.108 90)
 			(show_name no)
@@
 			)
 		)
-		(property "Value" "15k"
+		(property "Value" "4.7K"
 			(at 65.024 70.612 90)
 			(show_name no)
@@
 			)
 		)
-		(property "Value" "47k"
+		(property "Value" "47K"
 			(at 109.22 129.794 90)
 			(show_name no)
@@
 			)
 		)
-		(property "Value" "4.7k"
+		(property "Value" "4.7K"
 			(at 163.83 30.734 90)
 			(show_name no)
@@
 			)
 		)
-		(property "Value" "4.7k"
+		(property "Value" "4.7K"
 			(at 191.77 153.924 90)
 			(show_name no)
@@
 			)
 		)
-		(property "Value" "1.8k"
+		(property "Value" "1.8K"
 			(at 152.4 118.364 90)
 			(show_name no)
@@
 			)
 		)
-		(property "Value" "22k"
+		(property "Value" "22K"
 			(at 101.346 69.85 90)
 			(show_name no)
@@
 			)
 		)
-		(property "Value" "33k"
+		(property "Value" "33K"
 			(at 97.79 129.794 90)
 			(show_name no)
@@
 			)
 		)
-		(property "Value" "1.5k"
+		(property "Value" "1.5K"
 			(at 153.416 90.17 90)
 			(show_name no)
